File: OBDBaja/OBDBajaInterface/OBDBajaInterface.kicad_pcb (KiCad board)
At the start: 2 copper layers, 43.4 x 44.5 mm, 17 parts, among them J1 Conn_01x02, J10 Conn_01x03, J11 Conn_01x03, J12 Conn_01x03, J13 Conn_01x03, J14 Conn_01x03, J15 Conn_01x03, J16 Conn_01x04, J17 Conn_01x04, J2 Conn_01x05, J3 Conn_01x05, J4 Conn_01x01, J5 Conn_01x01, J6 Conn_01x03, J7 Conn_01x03, J8 Conn_01x03, J9 Conn_01x03

Commit message: Updated OBD Baja file organization
Parts:
- added U1: SN65HVD232, Package_SO:SOIC-8_3.9x4.9mm_P1.27mm, F.Cu at (104.2, 69.8)
Connections:
- J16 pad 1: Net-(J16-Pin_1) -> /D7
- J16 pad 2: Net-(J16-Pin_2) -> /D6
- J16 pad 3: Net-(J16-Pin_3) -> /A3
- J16 pad 4: Net-(J16-Pin_4) -> /A4
- J17 pad 1: Net-(J16-Pin_1) -> /D7
- J17 pad 2: Net-(J16-Pin_2) -> /D6
- J17 pad 3: Net-(J16-Pin_3) -> /A3
- J17 pad 4: Net-(J16-Pin_4) -> /A4
Changed lines of the file:
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@@
   (net 13 "+5V")
   (net 14 "GND")
-  (net 15 "Net-(J16-Pin_1)")
-  (net 16 "Net-(J16-Pin_2)")
-  (net 17 "Net-(J16-Pin_3)")
-  (net 18 "Net-(J16-Pin_4)")
+  (net 15 "unconnected-(U1-GND-Pad2)")
+  (net 16 "unconnected-(U1-VCC-Pad3)")
+  (net 17 "unconnected-(U1-NC-Pad5)")
+  (net 18 "unconnected-(U1-CANL-Pad6)")
+  (net 19 "unconnected-(U1-CANH-Pad7)")
+  (net 20 "unconnected-(U1-NC-Pad8)")
   (footprint "Connector_PinHeader_2.54mm:PinHeader_1x03_P2.54mm_Horizontal" (layer "F.Cu")
     (at 111.14 53.34 90)
@@
       (stroke (width 0.1) (type solid)) (layer "F.Fab"))
     (pad "1" thru_hole rect (at 0 0) (size 1.7 1.7) (drill 1) (layers "*.Cu" "*.Mask")
-      (net 15 "Net-(J16-Pin_1)") (pinfunction "Pin_1") (pintype "passive"))
+      (net 7 "/D7") (pinfunction "Pin_1") (pintype "passive"))
     (pad "2" thru_hole oval (at 0 2.54) (size 1.7 1.7) (drill 1) (layers "*.Cu" "*.Mask")
-      (net 16 "Net-(J16-Pin_2)") (pinfunction "Pin_2") (pintype "passive"))
+      (net 6 "/D6") (pinfunction "Pin_2") (pintype "passive"))
     (pad "3" thru_hole oval (at 0 5.08) (size 1.7 1.7) (drill 1) (layers "*.Cu" "*.Mask")
-      (net 17 "Net-(J16-Pin_3)") (pinfunction "Pin_3") (pintype "passive"))
+      (net 11 "/A3") (pinfunction "Pin_3") (pintype "passive"))
     (pad "4" thru_hole oval (at 0 7.62) (size 1.7 1.7) (drill 1) (layers "*.Cu" "*.Mask")
-      (net 18 "Net-(J16-Pin_4)") (pinfunction "Pin_4") (pintype "passive"))
+      (net 12 "/A4") (pinfunction "Pin_4") (pintype "passive"))
     (model "${KICAD6_3DMODEL_DIR}/Connector_PinHeader_2.54mm.3dshapes/PinHeader_1x04_P2.54mm_Vertical.wrl" hide
       (offset (xyz 0 0 0))
@@
       (net 14 "GND") (pinfunction "Pin_3") (pintype "passive"))
     (model "${KICAD6_3DMODEL_DIR}/Connector_PinHeader_2.54mm.3dshapes/PinHeader_1x03_P2.54mm_Vertical.wrl" hide
+      (offset (xyz 0 0 0))
+      (scale (xyz 1 1 1))
+      (rotate (xyz 0 0 0))
+    )
+  )
+  (footprint "Package_SO:SOIC-8_3.9x4.9mm_P1.27mm" (layer "F.Cu")
+    (at 104.205 69.85)
+    (descr "SOIC, 8 Pin (JEDEC MS-012AA, https://www.analog.com/media/en/package-pcb-resources/package/pkg_pdf/soic_narrow-r/r_8.pdf), generated with kicad-footprint-generator ipc_gullwing_generator.py")
+    (tags "SOIC SO")
+    (property "Sheetfile" "OBDBajaInterface.kicad_sch")
+    (property "Sheetname" "")
+    (property "ki_description" "CAN Bus Transceivers, 3.3V, 1Mbps, SOIC-8")
+    (property "ki_keywords" "can transeiver ti")
+    (attr smd)
+    (fp_text reference "U1" (at 0 -3.4) (layer "F.SilkS")
+        (effects (font (size 1 1) (thickness 0.15)))
+    )
+    (fp_text value "SN65HVD232" (at 0 3.4) (layer "F.Fab")
+        (effects (font (size 1 1) (thickness 0.15)))
+    )
+    (fp_text user "${REFERENCE}" (at 0 0) (layer "F.Fab")
+        (effects (font (size 0.98 0.98) (thickness 0.15)))
+    )
+    (fp_line (start 0 -2.56) (end -3.45 -2.56)
+      (stroke (width 0.12) (type solid)) (layer "F.SilkS"))
+    (fp_line (start 0 -2.56) (end 1.95 -2.56)
+      (stroke (width 0.12) (type solid)) (layer "F.SilkS"))
+    (fp_line (start 0 2.56) (end -1.95 2.56)
+      (stroke (width 0.12) (type solid)) (layer "F.SilkS"))
+    (fp_line (start 0 2.56) (end 1.95 2.56)
+      (stroke (width 0.12) (type solid)) (layer "F.SilkS"))
+    (fp_line (start -3.7 -2.7) (end -3.7 2.7)
+      (stroke (width 0.05) (type solid)) (layer "F.CrtYd"))
+    (fp_line (start -3.7 2.7) (end 3.7 2.7)
+      (stroke (width 0.05) (type solid)) (layer "F.CrtYd"))
+    (fp_line (start 3.7 -2.7) (end -3.7 -2.7)
+      (stroke (width 0.05) (type solid)) (layer "F.CrtYd"))
+    (fp_line (start 3.7 2.7) (end 3.7 -2.7)
+      (stroke (width 0.05) (type solid)) (layer "F.CrtYd"))
+    (fp_line (start -1.95 -1.475) (end -0.975 -2.45)
+      (stroke (width 0.1) (type solid)) (layer "F.Fab"))
+    (fp_line (start -1.95 2.45) (end -1.95 -1.475)
+      (stroke (width 0.1) (type solid)) (layer "F.Fab"))
+    (fp_line (start -0.975 -2.45) (end 1.95 -2.45)
+      (stroke (width 0.1) (type solid)) (layer "F.Fab"))
+    (fp_line (start 1.95 -2.45) (end 1.95 2.45)
+      (stroke (width 0.1) (type solid)) (layer "F.Fab"))
+    (fp_line (start 1.95 2.45) (end -1.95 2.45)
+      (stroke (width 0.1) (type solid)) (layer "F.Fab"))
+    (pad "1" smd roundrect (at -2.475 -1.905) (size 1.95 0.6) (layers "F.Cu" "F.Paste" "F.Mask") (roundrect_rratio 0.25)
+      (net 1 "/CRX") (pinfunction "D") (pintype "input"))
+    (pad "2" smd roundrect (at -2.475 -0.635) (size 1.95 0.6) (layers "F.Cu" "F.Paste" "F.Mask") (roundrect_rratio 0.25)
+      (net 15 "unconnected-(U1-GND-Pad2)") (pinfunction "GND") (pintype "power_in"))
+    (pad "3" smd roundrect (at -2.475 0.635) (size 1.95 0.6) (layers "F.Cu" "F.Paste" "F.Mask") (roundrect_rratio 0.25)
+      (net 16 "unconnected-(U1-VCC-Pad3)") (pinfunction "VCC") (pintype "power_in"))
+    (pad "4" smd roundrect (at -2.475 1.905) (size 1.95 0.6) (layers "F.Cu" "F.Paste" "F.Mask") (roundrect_rratio 0.25)
+      (net 2 "/CTX") (pinfunction "R") (pintype "output"))
+    (pad "5" smd roundrect (at 2.475 1.905) (size 1.95 0.6) (layers "F.Cu" "F.Paste" "F.Mask") (roundrect_rratio 0.25)
+      (net 17 "unconnected-(U1-NC-Pad5)") (pinfunction "NC") (pintype "no_connect"))
+    (pad "6" smd roundrect (at 2.475 0.635) (size 1.95 0.6) (layers "F.Cu" "F.Paste" "F.Mask") (roundrect_rratio 0.25)
+      (net 18 "unconnected-(U1-CANL-Pad6)") (pinfunction "CANL") (pintype "bidirectional"))
+    (pad "7" smd roundrect (at 2.475 -0.635) (size 1.95 0.6) (layers "F.Cu" "F.Paste" "F.Mask") (roundrect_rratio 0.25)
+      (net 19 "unconnected-(U1-CANH-Pad7)") (pinfunction "CANH") (pintype "bidirectional"))
+    (pad "8" smd roundrect (at 2.475 -1.905) (size 1.95 0.6) (layers "F.Cu" "F.Paste" "F.Mask") (roundrect_rratio 0.25)
+      (net 20 "unconnected-(U1-NC-Pad8)") (pinfunction "NC") (pintype "no_connect"))
+    (model "${KICAD6_3DMODEL_DIR}/Package_SO.3dshapes/SOIC-8_3.9x4.9mm_P1.27mm.wrl"
       (offset (xyz 0 0 0))
       (scale (xyz 1 1 1))
@@
       (stroke (width 0.1) (type solid)) (layer "B.Fab"))
     (pad "1" thru_hole rect (at 0 0 180) (size 1.7 1.7) (drill 1) (layers "*.Cu" "*.Mask")
-      (net 15 "Net-(J16-Pin_1)") (pinfunction "Pin_1") (pintype "passive"))
+      (net 7 "/D7") (pinfunction "Pin_1") (pintype "passive"))
     (pad "2" thru_hole oval (at 0 -2.54 180) (size 1.7 1.7) (drill 1) (layers "*.Cu" "*.Mask")
-      (net 16 "Net-(J16-Pin_2)") (pinfunction "Pin_2") (pintype "passive"))
+      (net 6 "/D6") (pinfunction "Pin_2") (pintype "passive"))
     (pad "3" thru_hole oval (at 0 -5.08 180) (size 1.7 1.7) (drill 1) (layers "*.Cu" "*.Mask")
-      (net 17 "Net-(J16-Pin_3)") (pinfunction "Pin_3") (pintype "passive"))
+      (net 11 "/A3") (pinfunction "Pin_3") (pintype "passive"))
     (pad "4" thru_hole oval (at 0 -7.62 180) (size 1.7 1.7) (drill 1) (layers "*.Cu" "*.Mask")
-      (net 18 "Net-(J16-Pin_4)") (pinfunction "Pin_4") (pintype "passive"))
+      (net 12 "/A4") (pinfunction "Pin_4") (pintype "passive"))
     (model "${KICAD6_3DMODEL_DIR}/Connector_PinSocket_2.54mm.3dshapes/PinSocket_1x04_P2.54mm_Vertical.wrl"
       (offset (xyz 0 0 0))

Commit message: Finished PCB and test enclosure
Parts:
- removed J3: Conn_01x05, Connector_PinSocket_2.54mm:PinSocket_1x05_P2.54mm_Horizontal
- added C1: 0.1u, Capacitor_SMD:C_0805_2012Metric_Pad1.18x1.45mm_HandSolder, F.Cu at (107.3, 62.0)
- added C2: 0.1u, Capacitor_SMD:C_0805_2012Metric_Pad1.18x1.45mm_HandSolder, F.Cu at (109.3, 62.0)
- added D1: PESD3V3L2BT,215, Package_TO_SOT_SMD:SOT-23, F.Cu at (122.0, 60.3)
- added G***: LOGO, OBDBaja:baja_logo, F.Cu at (108.1, 71.8)
- added J18: Conn_01x01, Connector_PinSocket_2.54mm:PinSocket_1x01_P2.54mm_Horizontal, F.Cu at (89.5, 55.4)
- added J19: Conn_01x04, Connector_PinHeader_2.54mm:PinHeader_1x04_P2.54mm_Horizontal, F.Cu at (125.8, 54.0)
- added MH3: MountingHole_3.2mm_M3, MountingHole:MountingHole_3.2mm_M3, F.Cu at (126.0, 46.4)
- added MH4: MountingHole_3.2mm_M3, MountingHole:MountingHole_3.2mm_M3, F.Cu at (126.0, 97.2)
- added R1: 120, Resistor_SMD:R_0805_2012Metric_Pad1.20x1.40mm_HandSolder, F.Cu at (119.0, 60.3)
- J2: value Conn_01x05 -> Conn_01x10; footprint Connector_PinSocket_2.54mm:PinSocket_1x05_P2.54mm_Horizontal -> Connector_PinSocket_2.54mm:PinSocket_1x10_P2.54mm_Horizontal
- moved U1 13.7 mm to (114.0, 60.3)
- moved J10 5.05 mm to (102.2, 57.1), turned to 90 degrees
- moved J1 3.20 mm to (89.5, 59.1)
- moved J2 2.46 mm to (89.5, 65.3)
- moved J5 0.38 mm to (89.5, 91.8)
- moved J4 0.38 mm to (89.5, 51.7)
Connections:
- U1 pad 1: /CRX -> /CTX
- U1 pad 2: unconnected-(U1-GND-Pad2) -> GND
- U1 pad 3: unconnected-(U1-VCC-Pad3) -> +3.3V
- U1 pad 4: /CTX -> /CRX
- U1 pad 6: unconnected-(U1-CANL-Pad6) -> /CAN_N
- U1 pad 7: unconnected-(U1-CANH-Pad7) -> /CAN_P
Routing:
- net +5V: track 0.00 -> 117.6 mm
- net /D6: track 0.00 -> 65.4 mm
- net /D7: track 0.00 -> 64.6 mm
- net /A3: track 0.00 -> 49.6 mm
- net /A4: track 0.00 -> 45.2 mm
- net /D5: track 0.00 -> 31.2 mm
- net /A2: track 0.00 -> 27.8 mm
- net /CRX: track 0.00 -> 23.5 mm
- net +3.3V: track 0.00 -> 22.3 mm
- net /CTX: track 0.00 -> 22.2 mm
- net /D4: track 0.00 -> 21.7 mm
- net /A1: track 0.00 -> 17.1 mm
- net /D3: track 0.00 -> 14.6 mm
- net /CAN_N: track 0.00 -> 9.59 mm
- net /CAN_P: track 0.00 -> 9.58 mm
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Other:
- board size 43.4 x 44.5 mm -> 43.4 x 58.4 mm
- board text added: "2023"
- board text added: "OBD Baja Interface Module"

Commit message: Finalized PCB Files and Gerbers for order
Routing:
- net +3.3V: track 22.3 -> 31.8 mm
- net /CRX: track 23.5 -> 30.0 mm
- net GND: track 0.89 -> 2.60 mm, vias 1 -> 2
- net /CTX: track 22.2 -> 23.4 mm
Other:
- board text added: "+"
- board text added: "-"
- board text added: "A3 A4 A0 A1 A2"
- board text added: "CAN BUS"
- board text added: "D"
- board text added: "D3 D4 D5 D6 D7"
- board text added: "H"
- board text added: "I/O"
- board text added: "JLCJLCJLCJLC"
- board text added: "L"
- board text added: "SD"
- board text removed: "2023"
