File: Previous Sensor Boards/BajaSensorBoard/BajaSensorBoard.kicad_pcb (KiCad board)
At the start: 2 copper layers, 47 x 33 mm, 23 parts, among them J1 ICSP, J2 POWER/CAN, J3 Conn_01x06, U1 ATtiny841-SS, U2 MCP25625-x-SS, Y1 CSTNE16M0VH3C000R0

Commit message: Reorganization
Connections:
- J1 pad 1: /MISO -> /STBY
- J1 pad 3: /SCK -> /USER0
- J1 pad 4: /MOSI -> /USER1
Routing:
- net /USER1: track 10.0 -> 33.8 mm, vias 0 -> 1
- net /USER0: track 15.4 -> 33.8 mm
- net /STBY: track 16.2 -> 29.6 mm
- net /MOSI: track 16.8 -> 8.48 mm, vias 1 -> 0
- net /MISO: track 20.4 -> 13.1 mm, vias 1 -> 0
- net /SCK: track 27.6 -> 22.9 mm, vias 1 -> 0
