File: BajaCAN/BajaCAN.kicad_sch (KiCad schematic)
At the start: 19 parts, among them J1 Conn_01x04, J2 ICSP, U1 AVR128DB32x-xPT, U2 MCP25625-x-SS, U3 MCP1603, Y1 OV-7604-C7, Y2 CSTNE16M0VH3C000R0

Commit message: Change to CAN FD transciever
Parts:
- removed U2: MCP25625-x-SS, Package_SO:SSOP-28_5.3x10.2mm_P0.65mm, symbol Interface_CAN_LIN:MCP25625-x-SS
- added C2: 0.1u, symbol Device:C_Small
- added J3: Conn_01x04, symbol Connector_Generic:Conn_01x04
- added U4: MCP251863T-H-SS, Package_SO:SSOP-28_5.3x10.2mm_P0.65mm, symbol Interface_CAN_LIN:MCP251863T-H-SS
Connections:
- net +5V: now also C2.1, U4.1 (VIO), U4.14 (VDD), U4.25 (VCC)
- net CAN_H: now also U4.4 (CANH)
- net CAN_L: now also U4.3 (CANL)
- net GND: now also C2.2, U4.22 (VSS), U4.24 (GND)
- net MCP_INT: now also U4.19 (~{INT})
- net MCP_STBY: now also U4.5 (STBY)
- net MISO0: now also U4.11 (SDO)
- net MOSI0: now also U4.10 (SDI)
- net RX0: now also J3.2 (Pin_2)
- net SCK0: now also U4.9 (SCK)
- net SCL0: now also J3.4 (Pin_4)
- net SDA0: now also J3.3 (Pin_3)
- net TX0: now also J3.1 (Pin_1)
- net ~{SS}0: now also U4.13 (~{CS})
- net at Y2.1: now also U4.21 (OSC1)
- net at Y2.3: now also U4.20 (OSC2)
- new net: U4.15 (TXCAN), U4.23 (TXD)
- new net: U4.16 (RXCAN), U4.28 (RXD)
- no-connect marks 7 -> 3
Other:
- moved on the sheet: C7, Y2
