File: Current Projects/BajaCAN/BajaCAN.kicad_pcb (KiCad board)
At the start: 2 copper layers, 65.5 x 71.6 mm, 49 parts, among them J1 348300801, J2 PROG, J3 348302004, J4 348302001, U1 AVR128DB32x-xRXB, U2 MCP1603, U3 MCP251863T-H-SS, Y1 OV-7604-C7, Y2 CSTNE20M0V530000R0

Commit message: Schematic Annotations (no board changes)
Connections:
- net /OSC1 renamed Net-(U3-OSC2)
- net /OSC2 renamed Net-(U3-OSC1)
Changed lines of the file:
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@@
 	(net 49 "/SDO")
 	(net 50 "/SCK")
-	(net 51 "/OSC2")
-	(net 52 "/RXD")
-	(net 53 "/TXD")
-	(net 54 "/OSC1")
+	(net 51 "/RXD")
+	(net 52 "/TXD")
+	(net 53 "Net-(U3-OSC1)")
+	(net 54 "Net-(U3-OSC2)")
 	(footprint "Connector_PinHeader_2.54mm:PinHeader_1x04_P2.54mm_Vertical"
 		(layer "F.Cu")
@@
 			(size 0.4 1.9)
 			(layers "F.Cu" "F.Mask" "F.Paste")
-			(net 51 "/OSC2")
+			(net 53 "Net-(U3-OSC1)")
 			(pinfunction "1")
 			(pintype "passive")
@@
 			(size 0.4 1.9)
 			(layers "F.Cu" "F.Mask" "F.Paste")
-			(net 54 "/OSC1")
+			(net 54 "Net-(U3-OSC2)")
 			(pinfunction "3")
 			(pintype "passive")
@@
 			(layers "F.Cu" "F.Mask" "F.Paste")
 			(roundrect_rratio 0.25)
-			(net 52 "/RXD")
+			(net 51 "/RXD")
 			(pinfunction "RXCAN")
 			(pintype "input")
@@
 			(layers "F.Cu" "F.Mask" "F.Paste")
 			(roundrect_rratio 0.25)
-			(net 54 "/OSC1")
+			(net 54 "Net-(U3-OSC2)")
 			(pinfunction "OSC2")
 			(pintype "output")
@@
 			(layers "F.Cu" "F.Mask" "F.Paste")
 			(roundrect_rratio 0.25)
-			(net 51 "/OSC2")
+			(net 53 "Net-(U3-OSC1)")
 			(pinfunction "OSC1")
 			(pintype "input")
@@
 			(layers "F.Cu" "F.Mask" "F.Paste")
 			(roundrect_rratio 0.25)
-			(net 52 "/RXD")
+			(net 51 "/RXD")
 			(pinfunction "RXD")
 			(pintype "output")
@@
 			(layers "F.Cu" "F.Mask" "F.Paste")
 			(roundrect_rratio 0.25)
-			(net 53 "/TXD")
+			(net 52 "/TXD")
 			(pinfunction "TXD")
 			(pintype "output")
@@
 			(layers "F.Cu" "F.Mask" "F.Paste")
 			(roundrect_rratio 0.25)
-			(net 53 "/TXD")
+			(net 52 "/TXD")
 			(pinfunction "TXCAN")
 			(pintype "output")
@@
 	)
 	(segment
-		(start 131.626 106.483)
-		(end 133.039 106.483)
-		(width 0.2032)
-		(layer "F.Cu")
-		(net 51)
-	)
-	(segment
-		(start 133.039 106.483)
-		(end 134.041 105.481)
-		(width 0.2032)
-		(layer "F.Cu")
-		(net 51)
-	)
-	(segment
-		(start 134.041 105.481)
-		(end 134.535 105.481)
-		(width 0.2032)
-		(layer "F.Cu")
-		(net 51)
-	)
-	(segment
 		(start 133.727238 103.305562)
 		(end 133.902676 103.481)
 		(width 0.2032)
 		(layer "F.Cu")
-		(net 52)
+		(net 51)
 	)
 	(segment
@@
 		(width 0.2032)
 		(layer "F.Cu")
-		(net 52)
+		(net 51)
 	)
 	(segment
@@
 		(width 0.2032)
 		(layer "F.Cu")
-		(net 52)
+		(net 51)
 	)
 	(segment
@@
 		(width 0.2032)
 		(layer "F.Cu")
-		(net 52)
+		(net 51)
 	)
 	(segment
@@
 		(width 0.2032)
 		(layer "F.Cu")
-		(net 52)
+		(net 51)
 	)
 	(segment
@@
 		(width 0.2032)
 		(layer "F.Cu")
-		(net 52)
+		(net 51)
 	)
 	(via
@@
 		(drill 0.254)
 		(layers "F.Cu" "B.Cu")
-		(net 52)
+		(net 51)
 	)
 	(via
@@
 		(drill 0.254)
 		(layers "F.Cu" "B.Cu")
-		(net 52)
+		(net 51)
 	)
 	(segment
@@
 		(width 0.2032)
 		(layer "B.Cu")
-		(net 52)
+		(net 51)
 	)
 	(segment
@@
 		(width 0.2032)
 		(layer "B.Cu")
-		(net 52)
+		(net 51)
 	)
 	(segment
@@
 		(width 0.2032)
 		(layer "F.Cu")
-		(net 53)
+		(net 52)
 	)
 	(segment
@@
 		(width 0.2032)
 		(layer "F.Cu")
-		(net 53)
+		(net 52)
 	)
 	(segment
@@
 		(width 0.2032)
 		(layer "F.Cu")
-		(net 53)
+		(net 52)
 	)
 	(segment
@@
 		(width 0.2032)
 		(layer "F.Cu")
-		(net 53)
+		(net 52)
 	)
 	(via
@@
 		(drill 0.254)
 		(layers "F.Cu" "B.Cu")
-		(net 53)
+		(net 52)
 	)
 	(via
@@
 		(drill 0.254)
 		(layers "F.Cu" "B.Cu")
-		(net 53)
+		(net 52)
 	)
 	(segment
@@
 		(width 0.2032)
 		(layer "B.Cu")
-		(net 53)
+		(net 52)
 	)
 	(segment
@@
 		(width 0.2032)
 		(layer "B.Cu")
-		(net 53)
+		(net 52)
 	)
 	(segment
@@
 		(width 0.2032)
 		(layer "B.Cu")
-		(net 53)
+		(net 52)
 	)
 	(segment
@@
 		(width 0.2032)
 		(layer "B.Cu")
+		(net 52)
+	)
+	(segment
+		(start 131.626 106.483)
+		(end 133.039 106.483)
+		(width 0.2032)
+		(layer "F.Cu")
+		(net 53)
+	)
+	(segment
+		(start 133.039 106.483)
+		(end 134.041 105.481)
+		(width 0.2032)
+		(layer "F.Cu")
+		(net 53)
+	)
+	(segment
+		(start 134.041 105.481)
+		(end 134.535 105.481)
+		(width 0.2032)
+		(layer "F.Cu")
 		(net 53)
 	)
