File: Current Projects/BajaCAN_HAT/BajaCAN_HAT.kicad_sch (KiCad schematic)
At the start: 2 parts, among them U1 MCP2518FD-xQBB, U2 MCP2518FD-xQBB

Commit message: Reset main
Parts:
- added D1, D2: SM24CANB-02HTG, SM24CANB02HTG, symbol SM24CANB:SM24CANB-02HTG
- added J1: Conn_02x20_Odd_Even, symbol Connector_Generic:Conn_02x20_Odd_Even
- added U3: Si8642ED-B-IS, Package_SO:SOIC-16W_7.5x10.3mm_P1.27mm, symbol Isolator:Si8642ED-B-IS
- added U4, U5: SN65HVD230, Package_SO:SOIC-8_3.9x4.9mm_P1.27mm, symbol Interface_CAN_LIN:SN65HVD230
- added U6, U7: RT9193-33GB, SOT-23-5_RIT, symbol RT9193-33GB:RT9193-33GB
Connections:
- new net: U3.15 (GND2), U3.9 (GND2)
- new net: U3.2 (GND1), U3.8 (GND1)
Other:
- note added: "Placeholder for 9x1 MCU controller pins"
- note added: "Placeholder for CAN Screw Nodes 2x"
- note added: "Placeholder for EVISUN B0505LS-1W"
- note added: "Raspberry PI General IO 40 pin connector"
- moved on the sheet: U1, U2

Commit message: Schematic additions: Power 3V3, CAN_0, CAN_1, Power Isolator. Todo: Digital Isolator, Interface, Mode Switch, Stack Config,Power 5V, CAN Tranciver
Parts:
- added U8: RFMM-0505S, RFMM_RCP, symbol RFMM-0505S:RFMM-0505S
Connections:
- net CE_1: now reaches J1.12 (Pin_12)
- net GND: now reaches J1.14 (Pin_14)
- net GND: now also J1.20 (Pin_20), J1.25 (Pin_25), J1.30 (Pin_30), J1.34 (Pin_34), J1.39 (Pin_39), J1.6 (Pin_6), J1.9 (Pin_9)
- net INT_1: now reaches J1.18 (Pin_18)
- net MOSI_0: now reaches J1.19 (Pin_19)
- net +5V: now reaches J1.2 (Pin_2)
- net +5V: now also J1.4 (Pin_4)
- net MISO_0: now reaches J1.21 (Pin_21)
- net INT_0: now reaches J1.22 (Pin_22)
- net SCLK_0: now reaches J1.23 (Pin_23)
- net CE_0: now reaches J1.24 (Pin_24)
- net MISO_1: now reaches J1.35 (Pin_35)
- net MOSI_1: now reaches J1.38 (Pin_38)
- net SCLK_1: now reaches J1.40 (Pin_40)
Other:
- note removed: "Placeholder for 9x1 MCU controller pins"
- note removed: "Placeholder for CAN Screw Nodes 2x"
- note removed: "Placeholder for EVISUN B0505LS-1W"
- note removed: "Raspberry PI General IO 40 pin connector"
